File: eagle/RemoteInterface/HendiRemoteInterface_v010.brd (EAGLE design)
At the start: 90.2 x 52.1 mm, 34 parts, among them IC1 MAX31865, IC2 MAX31865, U1 WeMos D1 mini, X1 EPG.0B.309.HLN, X2 EPG.0B.309.HLN, X3 MKDSN1,5/4-5,08, X6 MKDSN1,5/4-5,08

Commit message: Update HendiRemoteInterface_v010.brd
Routing:
- net N$9: track 12.9 -> 10.1 mm
Changed lines of the file:
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@@
 <wire x1="79.005" y1="33.39" x2="81.03" y2="33.39" width="0.3048" layer="1"/>
 <wire x1="77.785" y1="34.61" x2="79.005" y2="33.39" width="0.3048" layer="1"/>
-<wire x1="73.5" y1="21.43" x2="73.5" y2="22.7" width="0.3048" layer="1"/>
 <wire x1="73.5" y1="22.7" x2="73.34" y2="22.86" width="0.3048" layer="1"/>
-<wire x1="73.66" y1="17.145" x2="73.66" y2="21.27" width="0.4064" layer="1"/>
-<wire x1="73.66" y1="21.27" x2="73.5" y2="21.43" width="0.4064" layer="1"/>
+<wire x1="73.66" y1="17.145" x2="73.66" y2="22.54" width="0.4064" layer="1"/>
+<wire x1="73.66" y1="22.54" x2="73.5" y2="22.7" width="0.4064" layer="1"/>
 <wire x1="75.565" y1="34.61" x2="73.34" y2="34.61" width="0.4064" layer="1"/>
 <wire x1="73.34" y1="35.88" x2="73.34" y2="34.61" width="0.4064" layer="1"/>
@@
 <contactref element="R5" pad="1"/>
 <contactref element="EXT2" pad="A"/>
-<wire x1="42.225" y1="22.86" x2="37.78" y2="22.86" width="0.3048" layer="1"/>
-<wire x1="42.225" y1="22.86" x2="43.18" y2="21.905" width="0.3048" layer="1"/>
-<wire x1="44.23" y1="16.095" x2="45.085" y2="16.095" width="0.3048" layer="1"/>
-<wire x1="43.18" y1="21.905" x2="43.18" y2="17.145" width="0.3048" layer="1"/>
-<wire x1="43.18" y1="17.145" x2="44.23" y2="16.095" width="0.3048" layer="1"/>
+<wire x1="44.545" y1="16.095" x2="45.085" y2="16.095" width="0.3048" layer="1"/>
+<wire x1="37.78" y1="22.86" x2="44.545" y2="16.095" width="0.3048" layer="1"/>
 </signal>
 <signal name="N$10">
